File: reference_solution/board/board.kicad_sch (KiCad schematic)
At the start: 29 parts, among them J1 USB_B_Micro, J2 SWD/UART, SW1 BOOT0, SW2 BOOT0, U1 MIC5365-3.3YC5, U2 STM32F401CEUx, U3 LSM6DSM, Y1 8MHz

Commit message: finished layout
Parts:
- removed R1: 10k, Resistor_SMD:R_0603_1608Metric, symbol Device:R_Small
- added H1: logo, extraparts:auv_logo, symbol Mechanical:MountingHole
- C10, C11, C12, C13, C2, C3, C4, C6, C8, C9: footprint (none) -> Capacitor_SMD:C_0603_1608Metric
- J1: footprint (none) -> extraparts:USB_Micro-B_U254-05
- J2: footprint (none) -> Connector:Tag-Connect_TC2050-IDC-NL_2x05_P1.27mm_Vertical
- SW1: footprint (none) -> Button_Switch_SMD:SW_SPST_PTS810
- SW2: value BOOT0 -> USR; footprint (none) -> Button_Switch_SMD:SW_SPST_PTS810
- renumbered R2 to R1, R3 to R2, R4 to R3, R5 to R4, R6 to R5, R7 to R6
